File: 2019_Tiva_Breakout/2019_Tiva_Breakout.kicad_pcb (KiCad board)
At the start: 2 copper layers, 139.8 x 79.5 mm, 10 parts, among them U1 TM4C129E_Launchpad

Commit message: Updated silkscreen with required information
Parts:
- added G***: LOGO, MRDT_Silkscreens:z_sig_Patrick_Sanchez_15mmx5mm, F.Cu at (138.4, 94.7)
Other:
- board text added: "TIVA Breakout Board, Rev. 1 Mars Rover Design Team Missouri S&T, 2020 Patrick Sanchez"
