File: Tiva_Breakout_Hardware/Tiva_Breakout_Hardware-Box.sch (KiCad schematic (older format))
At the start: 6 parts, among them U1 TM4C129E_Launchpad

Commit message: In process of changing layout for smaller board
Parts:
- removed 12V_B2: Molex_SL_04, MRDT_Connectors:MOLEX_SL_04_Horizontal, symbol Tiva_Breakout_Hardware-rescue:Molex_SL_04-MRDT_Connectors
- removed Conn30V_L1, Conn30V_R1: Molex_SL_08, MRDT_Connectors:MOLEX_SL_08_Horizontal, symbol MRDT_Connectors:Molex_SL_08
- added 12V_Board: Molex_SL_04, symbol MRDT_Connectors:Molex_SL_04
- added ConnA1: Molex_SL_09, MRDT_Connectors:MOLEX_SL_09_Horizontal, symbol MRDT_Connectors:Molex_SL_09
- added ConnB1, ConnD1, ConnD2: Molex_SL_08, MRDT_Connectors:MOLEX_SL_08_Horizontal, symbol MRDT_Connectors:Molex_SL_08
- added ConnC2: Molex_SL_10, MRDT_Connectors:MOLEX_SL_10_Horizontal, symbol MRDT_Connectors:Molex_SL_10
- ConnC1: renamed from ConnPCH_C2; symbol Tiva_Breakout_Hardware-rescue:Molex_SL_10-MRDT_Connectors -> MRDT_Connectors:Molex_SL_10
- ConnIN1: symbol Tiva_Breakout_Hardware-rescue:Molex_SL_04-MRDT_Connectors -> MRDT_Connectors:Molex_SL_04
- U1: symbol Tiva_Breakout_Hardware-rescue:TM4C129E_Launchpad-MRDT_Shields -> MRDT_Shields:TM4C129E_Launchpad
Connections:
- wire segments 50 -> 99
- no-connect marks 46 -> 15
